File: Docs/PCB/v2/KiCad/CNC_Foamcutter_Control_Board.kicad_pcb (KiCad board)
At the start: 2 copper layers, 83.8 x 88.9 mm, 36 parts, among them J1 24V_In, J10 Conn_02x04_Odd_Even, J11 State_Pins, J12 SD_Header, J13 Drive_Enable_Header, J14 Drive_Enable_Switches, J15 I2C_Breakout_0, J16 I2C_Breakout_1, J17 GPIO, J18 Lvl_Shift_HV, J19 Lvl_Shift_LV, J2 Buck_In_24V, J3 Buck_In_GND, J4 Buck_Out_5V, J5 Buck_Out_GND, J6 Joy_Header, J7 Button_LED_Negatives, J8 Lvl_Shift_LV, J9 Lvl_Shift_HV, Q1 IRF3205, Q2 IRF3205, Q3 IRF3205, U1 Teensy4.1

Commit message: Cleaned up PCB v2, should be ready for ordering
Parts:
- moved J18 19.7 mm to (110.4, 61.2)
- moved J19 19.7 mm to (120.4, 60.6)
- moved J8 19.3 mm to (120.5, 80.9)
- moved J9 19.3 mm to (110.3, 80.9)
- moved J10 10.00 mm to (104.4, 113.3), turned to 180 degrees
- moved J16 1.00 mm to (151.8, 89.6)
Routing:
- net Net-(J11-Pin_1): track 0.00 -> 85.8 mm
- net Net-(J10-Pin_1): track 0.00 -> 63.2 mm
- net Net-(J10-Pin_3): track 0.00 -> 57.5 mm
- net Net-(J17-Pin_11): track 0.00 -> 48.6 mm
- net (no net): track 42.4 -> 0.00 mm
- net Net-(J11-Pin_2): track 19.4 -> 60.2 mm
- net Net-(J10-Pin_2): track 0.00 -> 39.7 mm
- net Net-(J10-Pin_4): track 0.00 -> 34.1 mm
- net Net-(J19-Pin_4): track 0.00 -> 30.9 mm
- net Net-(J17-Pin_5): track 55.2 -> 27.3 mm
- net Net-(J7-Pin_1): track 0.00 -> 27.2 mm
- net Net-(J7-Pin_2): track 0.00 -> 25.9 mm
- net Net-(J7-Pin_3): track 57.6 -> 38.6 mm
- net Net-(J10-Pin_5): track 26.7 -> 45.7 mm
- net Net-(J13-Pin_1): track 13.8 -> 30.4 mm
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Other:
- board text added: "2-Axis CNC Foamcutter Controller v2"
- board text removed: "2-Axis CNC Foamcutter Controller v1"
